File: apps/kbd-usb/kicad/usb_kb.kicad_sch (KiCad schematic)
At the start: 18 parts, among them J2 USB_A, Q2 Q_NPN_BCE, U1 ATmega16U2-A, Y1 Crystal

Commit message: apps/kbd-usb/kicad: update project
Signed-off-by: Krzysztof Witek <kwitek@kw-net.com>
Parts:
- removed MISO1: MISO, Connector_PinHeader_2.54mm:PinHeader_1x01_P2.54mm_Vertical, symbol Connector:Conn_01x01_Male
- removed MOSI1: MOSI, Connector_PinHeader_2.54mm:PinHeader_1x01_P2.54mm_Vertical, symbol Connector:Conn_01x01_Male
- removed RST1: RST, Connector_PinHeader_2.54mm:PinHeader_1x01_P2.54mm_Vertical, symbol Connector:Conn_01x01_Male
- removed SCK1: SCK, Connector_PinHeader_2.54mm:PinHeader_1x01_P2.54mm_Vertical, symbol Connector:Conn_01x01_Male
- added J?: UART, symbol Connector:Conn_01x02_Male
- added J?: Conn_02x03_Odd_Even, symbol Connector_Generic:Conn_02x03_Odd_Even
Connections:
- net MISO_IC: now also J?.1 (Pin_1)
- net MOSI_IC: now also J?.4 (Pin_4)
- net RST_IC: now also J?.5 (Pin_5)
- net SCK_IC: now also J?.3 (Pin_3)
- net at U1.7 (PD1): now also R10k2.2, U1.8 (PD2), J?.2 (Pin_2)
- net at U1.9 (PD3): now also J?.1 (Pin_1)
Changed lines of the file:
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@@
 (kicad_sch (version 20211123) (generator eeschema)
   (paper "A4")
+  (junction (at 99.06 80.01) (diameter 0) (color 0 0 0 0)
+  )
   (junction (at 60.96 29.21) (diameter 0) (color 0 0 0 0)
   )
@@
   (junction (at 58.42 100.33) (diameter 0) (color 0 0 0 0)
   )
+  (junction (at 95.885 80.01) (diameter 0) (color 0 0 0 0)
+  )
   (junction (at 175.26 55.88) (diameter 0) (color 0 0 0 0)
   )
@@
     (stroke (width 0) (type default) (color 0 0 0 0))
   )
+  (wire (pts (xy 95.885 80.01) (xy 99.06 80.01))
+    (stroke (width 0) (type default) (color 0 0 0 0))
+  )
+  (wire (pts (xy 95.885 77.47) (xy 95.885 80.01))
+    (stroke (width 0) (type default) (color 0 0 0 0))
+  )
   (wire (pts (xy 113.03 17.78) (xy 113.03 24.13))
     (stroke (width 0) (type default) (color 0 0 0 0))
   )
+  (wire (pts (xy 78.74 82.55) (xy 108.585 82.55))
+    (stroke (width 0) (type default) (color 0 0 0 0))
+  )
   (wire (pts (xy 60.96 17.78) (xy 60.96 29.21))
     (stroke (width 0) (type default) (color 0 0 0 0))
   )
+  (wire (pts (xy 108.585 82.55) (xy 108.585 77.47))
+    (stroke (width 0) (type default) (color 0 0 0 0))
+  )
   (wire (pts (xy 60.96 17.78) (xy 113.03 17.78))
     (stroke (width 0) (type default) (color 0 0 0 0))
@@
     (stroke (width 0) (type default) (color 0 0 0 0))
   )
-  (wire (pts (xy 78.74 80.01) (xy 99.06 80.01))
-    (stroke (width 0) (type default) (color 0 0 0 0))
-  )
   (wire (pts (xy 175.26 55.88) (xy 177.8 55.88))
     (stroke (width 0) (type default) (color 0 0 0 0))
@@
     (stroke (width 0) (type default) (color 0 0 0 0))
   )
+  (wire (pts (xy 106.045 80.01) (xy 106.045 74.93))
+    (stroke (width 0) (type default) (color 0 0 0 0))
+  )
   (wire (pts (xy 41.91 36.83) (xy 41.91 30.48))
     (stroke (width 0) (type default) (color 0 0 0 0))
@@
     (stroke (width 0) (type default) (color 0 0 0 0))
   )
+  (wire (pts (xy 106.045 74.93) (xy 108.585 74.93))
+    (stroke (width 0) (type default) (color 0 0 0 0))
+  )
   (wire (pts (xy 105.41 39.37) (xy 105.41 40.64))
     (stroke (width 0) (type default) (color 0 0 0 0))
@@
     (stroke (width 0) (type default) (color 0 0 0 0))
   )
+  (wire (pts (xy 99.06 80.01) (xy 106.045 80.01))
+    (stroke (width 0) (type default) (color 0 0 0 0))
+  )
   (wire (pts (xy 161.29 55.88) (xy 175.26 55.88))
     (stroke (width 0) (type default) (color 0 0 0 0))
@@
     (stroke (width 0) (type default) (color 0 0 0 0))
   )
+  (wire (pts (xy 78.74 80.01) (xy 95.885 80.01))
+    (stroke (width 0) (type default) (color 0 0 0 0))
+  )
   (wire (pts (xy 58.42 100.33) (xy 60.96 100.33))
+    (stroke (width 0) (type default) (color 0 0 0 0))
+  )
+  (wire (pts (xy 78.74 77.47) (xy 95.885 77.47))
     (stroke (width 0) (type default) (color 0 0 0 0))
   )
@@
     (effects (font (size 1.27 1.27)) (justify right bottom))
   )
-  (label "SCK_IC" (at 130.81 53.34 0)
-    (effects (font (size 1.27 1.27)) (justify left bottom))
+  (label "SCK_IC" (at 106.045 59.055 180)
+    (effects (font (size 1.27 1.27)) (justify right bottom))
   )
   (label "VCC" (at 111.76 105.41 0)
     (effects (font (size 1.27 1.27)) (justify left bottom))
   )
-  (label "MISO_IC" (at 110.49 59.69 0)
-    (effects (font (size 1.27 1.27)) (justify left bottom))
-  )
-  (label "RST_IC" (at 111.76 67.31 0)
-    (effects (font (size 1.27 1.27)) (justify left bottom))
-  )
-  (label "MOSI_IC" (at 130.81 60.96 0)
+  (label "MISO_IC" (at 106.045 56.515 180)
+    (effects (font (size 1.27 1.27)) (justify right bottom))
+  )
+  (label "RST_IC" (at 106.045 61.595 180)
+    (effects (font (size 1.27 1.27)) (justify right bottom))
+  )
+  (label "MOSI_IC" (at 118.745 59.055 0)
     (effects (font (size 1.27 1.27)) (justify left bottom))
   )
@@
     (pin "4")
   )
-  (symbol (lib_id "Connector:Conn_01x01_Male") (at 105.41 59.69 0) (unit 1)
-    (in_bom yes) (on_board yes) (fields_autoplaced)
-    (property "Reference" "MISO1" (id 0) (at 106.045 54.61 0))
-    (property "Value" "MISO" (id 1) (at 106.045 57.15 0))
-    (property "Footprint" "Connector_PinHeader_2.54mm:PinHeader_1x01_P2.54mm_Vertical" (id 2) (at 105.41 59.69 0)
-      (effects (font (size 1.27 1.27)) hide)
-    )
-    (property "Datasheet" "~" (id 3) (at 105.41 59.69 0)
-      (effects (font (size 1.27 1.27)) hide)
-    )
-    (pin "1")
-  )
   (symbol (lib_id "power:GND") (at 91.44 72.39 0) (unit 1)
     (in_bom yes) (on_board yes) (fields_autoplaced)
@@
     (pin "2")
   )
+  (symbol (lib_id "Connector:Conn_01x02_Male") (at 113.665 77.47 180) (unit 1)
+    (in_bom yes) (on_board yes) (fields_autoplaced)
+    (property "Reference" "J?" (id 0) (at 115.57 74.9299 0)
+      (effects (font (size 1.27 1.27)) (justify right))
+    )
+    (property "Value" "UART" (id 1) (at 115.57 77.4699 0)
+      (effects (font (size 1.27 1.27)) (justify right))
+    )
+    (property "Footprint" "" (id 2) (at 113.665 77.47 0)
+      (effects (font (size 1.27 1.27)) hide)
+    )
+    (property "Datasheet" "~" (id 3) (at 113.665 77.47 0)
+      (effects (font (size 1.27 1.27)) hide)
+    )
+    (pin "1")
+    (pin "2")
+  )
   (symbol (lib_id "alarm-rescue:R") (at 99.06 76.2 0) (unit 1)
     (in_bom yes) (on_board yes)
@@
     (pin "2")
   )
-  (symbol (lib_id "Connector:Conn_01x01_Male") (at 125.73 53.34 0) (unit 1)
-    (in_bom yes) (on_board yes) (fields_autoplaced)
-    (property "Reference" "SCK1" (id 0) (at 126.365 48.26 0))
-    (property "Value" "SCK" (id 1) (at 126.365 50.8 0))
-    (property "Footprint" "Connector_PinHeader_2.54mm:PinHeader_1x01_P2.54mm_Vertical" (id 2) (at 125.73 53.34 0)
-      (effects (font (size 1.27 1.27)) hide)
-    )
-    (property "Datasheet" "~" (id 3) (at 125.73 53.34 0)
-      (effects (font (size 1.27 1.27)) hide)
-    )
-    (pin "1")
-  )
   (symbol (lib_id "power:GND") (at 58.42 100.33 0) (unit 1)
     (in_bom yes) (on_board yes) (fields_autoplaced)
@@
     (pin "1")
   )
-  (symbol (lib_id "Connector:Conn_01x01_Male") (at 106.68 67.31 0) (unit 1)
-    (in_bom yes) (on_board yes)
-    (property "Reference" "RST1" (id 0) (at 107.315 62.23 0))
-    (property "Value" "RST" (id 1) (at 107.315 64.77 0))
-    (property "Footprint" "Connector_PinHeader_2.54mm:PinHeader_1x01_P2.54mm_Vertical" (id 2) (at 106.68 67.31 0)
-      (effects (font (size 1.27 1.27)) hide)
-    )
-    (property "Datasheet" "~" (id 3) (at 106.68 67.31 0)
-      (effects (font (size 1.27 1.27)) hide)
-    )
-    (pin "1")
-  )
   (symbol (lib_id "alarm-rescue:GND") (at 20.32 31.75 180) (unit 1)
     (in_bom yes) (on_board yes)
@@
     (pin "2")
   )
-  (symbol (lib_id "Connector:Conn_01x01_Male") (at 125.73 60.96 0) (unit 1)
-    (in_bom yes) (on_board yes)
-    (property "Reference" "MOSI1" (id 0) (at 126.365 55.88 0))
-    (property "Value" "MOSI" (id 1) (at 126.365 58.42 0))
-    (property "Footprint" "Connector_PinHeader_2.54mm:PinHeader_1x01_P2.54mm_Vertical" (id 2) (at 125.73 60.96 0)
-      (effects (font (size 1.27 1.27)) hide)
-    )
-    (property "Datasheet" "~" (id 3) (at 125.73 60.96 0)
-      (effects (font (size 1.27 1.27)) hide)
-    )
-    (pin "1")
-  )
   (symbol (lib_id "alarm-rescue:C") (at 20.32 35.56 0) (unit 1)
     (in_bom yes) (on_board yes)
@@
     (pin "1")
     (pin "2")
+  )
+  (symbol (lib_id "Connector_Generic:Conn_02x03_Odd_Even") (at 111.125 59.055 0) (unit 1)
+    (in_bom yes) (on_board yes) (fields_autoplaced)
+    (property "Reference" "J?" (id 0) (at 112.395 50.165 0))
+    (property "Value" "Conn_02x03_Odd_Even" (id 1) (at 112.395 52.705 0))
+    (property "Footprint" "" (id 2) (at 111.125 59.055 0)
+      (effects (font (size 1.27 1.27)) hide)
+    )
+    (property "Datasheet" "~" (id 3) (at 111.125 59.055 0)
+      (effects (font (size 1.27 1.27)) hide)
+    )
+    (pin "1")
+    (pin "2")
+    (pin "3")
+    (pin "4")
+    (pin "5")
+    (pin "6")
   )
   (sheet_instances
@@
       (reference "J2") (unit 1) (value "USB_A") (footprint "Connector_USB:USB_A_CNCTech_1001-011-01101_Horizontal")
     )
+    (path "/5a86e257-c952-407c-b2eb-3702a2156af1"
+      (reference "J?") (unit 1) (value "UART") (footprint "")
+    )
+    (path "/e338f1f3-cb85-47f5-8320-4af42ae65ea1"
+      (reference "J?") (unit 1) (value "Conn_02x03_Odd_Even") (footprint "")
+    )
     (path "/4f8dcdaa-eb04-41d3-8ccc-be8d02100ac3"
       (reference "LED1") (unit 1) (value "LED") (footprint "LED_THT:LED_D5.0mm")
     )
-    (path "/327b460e-b23b-4a49-9d27-5421e64533cd"
-      (reference "MISO1") (unit 1) (value "MISO") (footprint "Connector_PinHeader_2.54mm:PinHeader_1x01_P2.54mm_Vertical")
-    )
-    (path "/db607efe-93f3-4c97-9567-26eeb0ad9c9f"
-      (reference "MOSI1") (unit 1) (value "MOSI") (footprint "Connector_PinHeader_2.54mm:PinHeader_1x01_P2.54mm_Vertical")
-    )
     (path "/1e75a993-db82-4683-a8f3-99d9c5f521c2"
       (reference "Q2") (unit 1) (value "Q_NPN_BCE") (footprint "Package_TO_SOT_THT:TO-92")
@@
       (reference "R22_1") (unit 1) (value "R22") (footprint "Resistor_SMD:R_0805_2012Metric")
     )
-    (path "/c9d0c5bc-357a-4823-a8ac-039d63c9a587"
-      (reference "RST1") (unit 1) (value "RST") (footprint "Connector_PinHeader_2.54mm:PinHeader_1x01_P2.54mm_Vertical")
-    )
-    (path "/6ffb56da-ff35-4cb5-8efa-ee5f4bcc4627"
-      (reference "SCK1") (unit 1) (value "SCK") (footprint "Connector_PinHeader_2.54mm:PinHeader_1x01_P2.54mm_Vertical")
-    )
     (path "/2e0251dd-446f-46f7-a5c9-99c221e4a8c3"
