File: apps/kbd-usb/kbd-usb-remote-ctl/kicad/usb_kb_transmitter.kicad_pcb (KiCad board)
At the start: 2 copper layers, 30.1 x 53 mm, 15 parts, among them J1 Conn_01x02_Female, J6 SYN115, Q1 Q_NPN_BEC, Q2 Q_NPN_BEC, Q3 Q_NPN_BEC, SW1 SW_MEC_5E, SW2 SW_MEC_5E, SW3 SW_MEC_5E, U1 ATtiny85-20P

Commit message: apps/kbd-usb/kicad: update project
Signed-off-by: Krzysztof Witek <kwitek@kw-net.com>
Parts:
- removed Q1, Q2, Q3: Q_NPN_BEC, Package_TO_SOT_SMD:SOT-23-3
- removed R1, R2, R3: R4.7k, Resistor_SMD:R_0805_2012Metric
- removed SW2, SW3: SW_MEC_5E, Button_Switch_THT:SW_PUSH-12mm
- added RF-TX1: CONN_01X03, Connector_PinHeader_2.54mm:PinHeader_1x03_P2.54mm_Vertical, F.Cu at (137.1, 50.3)
- moved U1 24.2 mm to (120.7, 65.6)
- moved R10k_1 17.2 mm to (115.6, 66.9), turned to 90 degrees
- moved SW1 14.8 mm to (131.4, 44.7)
Connections:
- J6 pad 2: /GND_P -> GND
- J6 pad 4: +3.3V -> /VCC
- R10k1 pad 1: Net-(LED1-Pad2) -> Net-(U1-Pad7)
- R10k1 pad 2: /LED -> Net-(LED1-Pad2)
- R10k_1 pad 1: +3.3V -> /VCC
- SW1 pad 1: Net-(R1-Pad2) -> /VCC
- U1 pad 2: Net-(R2-Pad1) -> unconnected-(U1-Pad2)
- U1 pad 4: /GND_P -> GND
- U1 pad 5: Net-(R1-Pad1) -> unconnected-(U1-Pad5)
- U1 pad 6: Net-(R3-Pad1) -> unconnected-(U1-Pad6)
- U1 pad 7: /LED -> Net-(U1-Pad7)
- U1 pad 8: +3.3V -> /VCC
Routing:
- net +3.3V: track 95.0 -> 0.00 mm
- net /GND_P: track 80.8 -> 0.00 mm
- net GND: track 74.0 -> 0.00 mm
- net Net-(R3-Pad1): track 49.0 -> 0.00 mm
- net Net-(R1-Pad1): track 40.1 -> 0.00 mm, vias 1 -> 0
- net /T: track 38.4 -> 0.00 mm
- net Net-(R2-Pad1): track 34.9 -> 0.00 mm, vias 2 -> 0
- net /LED: track 32.7 -> 0.00 mm
- net Net-(R1-Pad2): track 17.1 -> 0.00 mm
- net Net-(R3-Pad2): track 16.3 -> 0.00 mm
- net Net-(R2-Pad2): track 16.3 -> 0.00 mm
- net Net-(R10k_1-Pad2): track 10.3 -> 0.00 mm, vias 1 -> 0
- net Net-(LED1-Pad2): track 7.14 -> 0.00 mm

Commit message: apps/kbd-usb/kbd-usb-remote-ctl: update kicad projet
Signed-off-by: Krzysztof Witek <kwitek@kw-net.com>
Parts:
- removed RF-TX1: CONN_01X03, Connector_PinHeader_2.54mm:PinHeader_1x03_P2.54mm_Vertical
- R10k1, R10k_1: footprint Resistor_SMD:R_0805_2012Metric -> Resistor_THT:R_Axial_DIN0204_L3.6mm_D1.6mm_P7.62mm_Horizontal
- moved R10k_1 17.4 mm to (112.1, 84.0), turned to 0 degrees
- moved R10k1 2.90 mm to (112.9, 55.8), turned to 90 degrees
Routing:
- net /VCC: track 0.00 -> 68.2 mm
- net GND: track 0.00 -> 49.1 mm
- net +3.3V: track 0.00 -> 30.7 mm
- net Net-(R10k_1-Pad2): track 0.00 -> 18.8 mm
- net /T: track 0.00 -> 18.2 mm
- net Net-(R10k1-Pad1): track 0.00 -> 12.7 mm
- net Net-(LED1-Pad2): track 0.00 -> 3.45 mm
Other:
- board text added: "KBD TX Krzysztof Witek v0.1 07/2024"
- board text added: "KW KBD USB Remote V0.1"
- board text removed: "KW KBD USB Remote V1.0"
