File: apps/kbd-usb/kbd-usb-remote-ctl/kicad/usb_kb_transmitter.kicad_sch (KiCad schematic)
At the start: 15 parts, among them J1 Conn_01x02_Female, J6 SYN115, Q1 Q_NPN_BEC, Q2 Q_NPN_BEC, Q3 Q_NPN_BEC, SW1 SW_MEC_5E, SW2 SW_MEC_5E, SW3 SW_MEC_5E, U1 ATtiny85-20P

Commit message: apps/kbd-usb/kicad: update project
Signed-off-by: Krzysztof Witek <kwitek@kw-net.com>
Parts:
- removed Q1, Q2, Q3: Q_NPN_BEC, Package_TO_SOT_SMD:SOT-23-3, symbol Device:Q_NPN_BEC
- removed R1, R2, R3: R4.7k, Resistor_SMD:R_0805_2012Metric, symbol Device:R
- removed SW2, SW3: SW_MEC_5E, Button_Switch_THT:SW_PUSH-12mm, symbol Switch:SW_MEC_5E
- added RF-TX1: CONN_01X03, Connector_PinHeader_2.54mm:PinHeader_1x03_P2.54mm_Vertical, symbol alarm_module1-rescue:CONN_01X03
Connections:
- net GND_P is gone; now on net GND: J6.2 (Pin_2), U1.4 (GND)
- net +3.3V: no longer J6.4 (Pin_4), R10k_1.1, U1.8 (VCC)
- net GND: now also RF-TX1.3 (P3)
- net T: now also RF-TX1.1 (P1)
- net at R10k1.1: now also U1.7 (PB2); no longer LED1.2 (A)
- net VCC: now reaches SW1.1
- net VCC: now also J6.4 (Pin_4), R10k_1.1, U1.8 (VCC), RF-TX1.2 (P2)
- net LED: no longer names the net of R10k1.2
- net LED: now also LED1.2 (A); no longer U1.7 (PB2)
Other:
- moved on the sheet: R10k1

Commit message: apps/kbd-usb/kbd-usb-remote-ctl: update kicad projet
Signed-off-by: Krzysztof Witek <kwitek@kw-net.com>
Parts:
- removed RF-TX1: CONN_01X03, Connector_PinHeader_2.54mm:PinHeader_1x03_P2.54mm_Vertical, symbol alarm_module1-rescue:CONN_01X03
- R10k1, R10k_1: footprint Resistor_SMD:R_0805_2012Metric -> Resistor_THT:R_Axial_DIN0204_L3.6mm_D1.6mm_P7.62mm_Horizontal
Changed lines of the file:
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@@
     (stroke (width 0) (type default) (color 0 0 0 0))
-  )
-  (label "T" (at 181.61 109.22 180)
-    (effects (font (size 1.27 1.27)) (justify right bottom))
   )
   (label "VCC" (at 111.76 67.31 180)
@@
   )
   (label "VCC" (at 127 95.25 270)
-    (effects (font (size 1.27 1.27)) (justify right bottom))
-  )
-  (label "VCC" (at 181.61 111.76 180)
     (effects (font (size 1.27 1.27)) (justify right bottom))
   )
@@
     (property "Reference" "R10k1" (id 0) (at 153.162 111.76 90))
     (property "Value" "R10k" (id 1) (at 151.13 111.76 90))
-    (property "Footprint" "Resistor_SMD:R_0805_2012Metric" (id 2) (at 149.352 111.76 90)
+    (property "Footprint" "Resistor_THT:R_Axial_DIN0204_L3.6mm_D1.6mm_P7.62mm_Horizontal" (id 2) (at 149.352 111.76 90)
       (effects (font (size 1.27 1.27)) hide)
     )
@@
     (pin "1")
     (pin "2")
-  )
-  (symbol (lib_id "alarm_module1-rescue:CONN_01X03") (at 186.69 111.76 0) (unit 1)
-    (in_bom yes) (on_board yes)
-    (property "Reference" "RF-TX1" (id 0) (at 186.69 106.68 0))
-    (property "Value" "CONN_01X03" (id 1) (at 189.23 111.76 90))
-    (property "Footprint" "Connector_PinHeader_2.54mm:PinHeader_1x03_P2.54mm_Vertical" (id 2) (at 186.69 111.76 0)
-      (effects (font (size 1.27 1.27)) hide)
-    )
-    (property "Datasheet" "" (id 3) (at 186.69 111.76 0))
-    (pin "1")
-    (pin "2")
-    (pin "3")
   )
   (symbol (lib_id "power:GND") (at 111.76 97.79 0) (unit 1)
@@
     (property "Reference" "R10k_1" (id 0) (at 124.968 91.44 90))
     (property "Value" "R10k" (id 1) (at 127 91.44 90))
-    (property "Footprint" "Resistor_SMD:R_0805_2012Metric" (id 2) (at 128.778 91.44 90)
+    (property "Footprint" "Resistor_THT:R_Axial_DIN0204_L3.6mm_D1.6mm_P7.62mm_Horizontal" (id 2) (at 128.778 91.44 90)
       (effects (font (size 1.27 1.27)) hide)
     )
@@
     (pin "3")
     (pin "4")
-  )
-  (symbol (lib_id "alarm_module1-rescue:GND") (at 181.61 114.3 270) (unit 1)
-    (in_bom yes) (on_board yes)
-    (property "Reference" "#PWR0104" (id 0) (at 175.26 114.3 0)
-      (effects (font (size 1.27 1.27)) hide)
-    )
-    (property "Value" "GND" (id 1) (at 177.8 114.3 0))
-    (property "Footprint" "" (id 2) (at 181.61 114.3 0))
-    (property "Datasheet" "" (id 3) (at 181.61 114.3 0))
-    (pin "1")
   )
   (symbol (lib_id "MCU_Microchip_ATtiny:ATtiny85-20P") (at 111.76 82.55 0) (unit 1)
@@
       (reference "#PWR0103") (unit 1) (value "GND") (footprint "")
     )
-    (path "/abb774bb-ea31-4fa1-a062-1e92376cfb7d"
-      (reference "#PWR0104") (unit 1) (value "GND") (footprint "")
-    )
     (path "/2d2338f3-bd59-458c-81fe-a7323afff612"
       (reference "#PWR0110") (unit 1) (value "+3.3V") (footprint "")
@@
     )
     (path "/595b9837-eeb3-44a2-9b43-69785b4ce2e2"
-      (reference "R10k1") (unit 1) (value "R10k") (footprint "Resistor_SMD:R_0805_2012Metric")
+      (reference "R10k1") (unit 1) (value "R10k") (footprint "Resistor_THT:R_Axial_DIN0204_L3.6mm_D1.6mm_P7.62mm_Horizontal")
     )
     (path "/6c7d47ce-32dd-491d-9871-34b32af18853"
-      (reference "R10k_1") (unit 1) (value "R10k") (footprint "Resistor_SMD:R_0805_2012Metric")
-    )
-    (path "/6268f123-e679-4f4a-bee7-dd8dfff9ca17"
-      (reference "RF-TX1") (unit 1) (value "CONN_01X03") (footprint "Connector_PinHeader_2.54mm:PinHeader_1x03_P2.54mm_Vertical")
+      (reference "R10k_1") (unit 1) (value "R10k") (footprint "Resistor_THT:R_Axial_DIN0204_L3.6mm_D1.6mm_P7.62mm_Horizontal")
     )
     (path "/a339698c-cf34-415f-b408-d8c9ae3f9b63"
